Commit message: Got the chassis raised and reoriented in rviz.

File: terraflight_description/urdf/terraflight.urdf.xacro (robot description, xacro)
@@ -1,20 +1,22 @@
 <?xml version="1.0" ?>
 <robot name="terraflight" xmlns:xacro="http://wiki.ros.org/wiki/xacro">
-<material name="purple">
-    <color rgba="0.3 0.16 0.52 1.0"/>
+<material name="grey">
+    <color rgba="0.7529 0.7529 0.7529 1.0"/>
 </material>
+<!-- Once I get a map/odom fixed frame (which is fixed to 0,0,0), I will want to both make the base_footprint directly underneath
+the chassis, and also offset the chassis spawning location -->
 <link name="base_footprint"/>
 <joint name="base_joint" type="fixed">
     <parent link="base_footprint"/>
     <child link="chassis"/>
-    <origin xyz="0.0 0.0 0.0" rpy="0 0 0"/>
+    <origin xyz="0.254 0.0 0.1226125" rpy="0 0 3.141592653589"/>
 </joint>
 <link name="chassis">
     <visual>
-        <origin xyz="1.0 1.0 1.0" rpy="0 0 0"/>
+        <origin xyz="0 0 0" rpy="0 0 0"/>
         <geometry>
             <mesh filename="package://terraflight_description/meshes/chassis.stl" scale="1 1 1"/>
         </geometry>
-        <material name="purple" />
+        <material name="grey" />
     </visual>
 </link>

Commit message: Got chassis set up in Rviz Fixed world frame and base footprint are good, too

File: terraflight_description/urdf/terraflight.urdf.xacro (robot description, xacro)
@@ -4,11 +4,9 @@
     <color rgba="0.7529 0.7529 0.7529 1.0"/>
 </material>
-<!-- Once I get a map/odom fixed frame (which is fixed to 0,0,0), I will want to both make the base_footprint directly underneath
-the chassis, and also offset the chassis spawning location -->
 <link name="base_footprint"/>
 <joint name="base_joint" type="fixed">
     <parent link="base_footprint"/>
     <child link="chassis"/>
-    <origin xyz="0.254 0.0 0.1226125" rpy="0 0 3.141592653589"/>
+    <origin xyz="0 0 0.1226125" rpy="0 0 3.141592653589"/>
 </joint>
 <link name="chassis">

Commit message: Added joint state publisher node so continuous joint wheel shows up

File: terraflight_description/urdf/terraflight.urdf.xacro (robot description, xacro)
@@ -3,4 +3,7 @@
 <material name="grey">
     <color rgba="0.7529 0.7529 0.7529 1.0"/>
+</material>
+<material name="dark">
+    <color rgba="0.2 0.2 0.2 1.0"/>
 </material>
 <link name="base_footprint"/>
@@ -19,3 +22,18 @@
     </visual>
 </link>
+<joint name="front_left_joint" type="continuous">
+    <parent link="chassis"/>
+    <child link="front_left_wheel"/>
+    <origin xyz="0 0 0"/>
+    <axis xyz="0 1 0"/>
+</joint>
+<link name="front_left_wheel">
+    <visual>
+        <origin xyz="0 0 0" rpy="0 0 0"/>
+        <geometry>
+            <mesh filename="package://terraflight_description/meshes/front_left_wheel.stl" scale="1 1 1"/>
+        </geometry>
+        <material name="dark"/>
+    </visual>
+</link>
 </robot>

Commit message: Got front left wheel on in rviz About as close positioning as I am going to get

File: terraflight_description/urdf/terraflight.urdf.xacro (robot description, xacro)
@@ -25,10 +25,10 @@
     <parent link="chassis"/>
     <child link="front_left_wheel"/>
-    <origin xyz="0 0 0"/>
+    <origin xyz="0 -.3433115 -0.0427975"/>
     <axis xyz="0 1 0"/>
 </joint>
 <link name="front_left_wheel">
     <visual>
-        <origin xyz="0 0 0" rpy="0 0 0"/>
+        <origin xyz="0 0 0" rpy="1.5708 0 0"/>
         <geometry>
             <mesh filename="package://terraflight_description/meshes/front_left_wheel.stl" scale="1 1 1"/>

Commit message: All 4 wheels on URDF still need to do collision and intertia

File: terraflight_description/urdf/terraflight.urdf.xacro (robot description, xacro)
@@ -37,3 +37,48 @@
     </visual>
 </link>
+<joint name="back_left_joint" type="continuous">
+    <parent link="chassis"/>
+    <child link="back_left_wheel"/>
+    <origin xyz=".4826 -.3433115 -0.0427975"/>
+    <axis xyz="0 1 0"/>
+</joint>
+<link name="back_left_wheel">
+    <visual>
+        <origin xyz="0 0 0" rpy="1.5708 0 0"/>
+        <geometry>
+            <mesh filename="package://terraflight_description/meshes/back_left_wheel.stl" scale="1 1 1"/>
+        </geometry>
+        <material name="dark"/>
+    </visual>
+</link>
+<joint name="front_right_joint" type="continuous">
+    <parent link="chassis"/>
+    <child link="front_right_wheel"/>
+    <origin xyz="0 .3433115 -0.0427975"/>
+    <axis xyz="0 1 0"/>
+</joint>
+<link name="front_right_wheel">
+    <visual>
+        <origin xyz="0 0 0" rpy="-1.5708 0 0"/>
+        <geometry>
+            <mesh filename="package://terraflight_description/meshes/front_right_wheel.stl" scale="1 1 1"/>
+        </geometry>
+        <material name="dark"/>
+    </visual>
+</link>
+<joint name="back_right_joint" type="continuous">
+    <parent link="chassis"/>
+    <child link="back_right_wheel"/>
+    <origin xyz=".4826 .3433115 -0.0427975"/>
+    <axis xyz="0 1 0"/>
+</joint>
+<link name="back_right_wheel">
+    <visual>
+        <origin xyz="0 0 0" rpy="1.5708 0 0"/>
+        <geometry>
+            <mesh filename="package://terraflight_description/meshes/back_right_wheel.stl" scale="1 1 1"/>
+        </geometry>
+        <material name="dark"/>
+    </visual>
+</link>
 </robot>

Commit message: TEST ODOM works
obviously this is not the optimal solution, but for indoor flat areas, it works

could use a little more tuning

File: terraflight_description/urdf/terraflight.urdf.xacro (robot description, xacro)
@@ -11,5 +11,5 @@
     <parent link="base_footprint"/>
     <child link="chassis"/>
-    <origin xyz="0 0 0.1226125" rpy="0 0 3.141592653589"/>
+    <origin xyz="0.254 0 0.1226125" rpy="0 0 3.141592653589"/>
 </joint>
 <link name="chassis">

Commit message: updated frames in urdf

File: terraflight_description/urdf/terraflight.urdf.xacro (robot description, xacro)
@@ -10,6 +10,19 @@
 <joint name="base_joint" type="fixed">
     <parent link="base_footprint"/>
+    <child link="base_link"/>
+    <origin xyz="0 0 0.1226125" rpy="0 0 3.141592653589"/>
+    <!-- x 0.254 -->
+</joint>
+<link name="base_link"/>
+<joint name="base_link_to_laser" type="fixed">
+    <parent link="base_link"/>
+    <child link="laser"/>
+    <origin xyz="0.05 0 0.2" rpy="0 0 3.141592"/>
+</joint>
+<link name="laser"/>
+<joint name="base_link_to_chassis" type="fixed">
+    <parent link="base_link"/>
     <child link="chassis"/>
-    <origin xyz="0.254 0 0.1226125" rpy="0 0 3.141592653589"/>
+    <origin xyz="0 0 0"/>
 </joint>
 <link name="chassis">

Commit message: testing odom

File: terraflight_description/urdf/terraflight.urdf.xacro (robot description, xacro)
@@ -11,5 +11,5 @@
     <parent link="base_footprint"/>
     <child link="base_link"/>
-    <origin xyz="0 0 0.1226125" rpy="0 0 3.141592653589"/>
+    <origin xyz="0.254 0 0.1226125" rpy="0 0 3.141592653589"/>
     <!-- x 0.254 -->
 </joint>

Commit message: Updated rviz config and urdf

File: terraflight_description/urdf/terraflight.urdf.xacro (robot description, xacro)
@@ -18,5 +18,5 @@
     <parent link="base_link"/>
     <child link="laser"/>
-    <origin xyz="0.05 0 0.2" rpy="0 0 3.141592"/>
+    <origin xyz="0.05 0 0.2" rpy="3.141592 0 3.141592"/>
 </joint>
 <link name="laser"/>
